Commit message: arm configured and working

File: public/urdf/arm/arm.urdf (robot description, URDF)
Before this commit: robot arm, 6 links, 5 joints
Links:
- link a_link: geometry visual mesh filename=../meshes/arm_a_fix.dae
- link c_link: geometry visual mesh filename=../meshes/arm_c_fix.dae
- link d_link: geometry visual mesh filename=../meshes/arm_d_fix.dae
- link e_link: geometry visual mesh filename=../meshes/arm_e_fix.dae
Joints:
- joint a_joint: origin xyz=19.923 20.023 54.02 rpy=0 0 0 -> xyz=3.4348 -0.0005 4.9028 rpy=0 0 0
- joint b_joint: origin xyz=0 0 0 rpy=0 0 0 -> xyz=53.4363 0.0005 0.9052 rpy=0 0 0
- joint base_link_joint: limit lower=0 upper=20 effort=30 velocity=1 -> lower=-40 upper=0 effort=30 velocity=1; origin xyz=0 -10 0 rpy=0 0 0 -> xyz=16.4882 20.0235 49.1172 rpy=0 0 0
- joint c_joint: origin xyz=0 0 0 rpy=0 0 0 -> xyz=54.6037 0 8.8594 rpy=0 0 0
- joint d_joint: origin xyz=0 0 0 rpy=0 0 0 -> xyz=4.488 0 0 rpy=0 0 0

Commit message: full rover done

File: public/urdf/arm/arm.urdf (robot description, URDF)
Before this commit: robot arm, 6 links, 5 joints
Links:
- added link arm_gripper_link; visual mesh filename=../meshes/arm_gripper_fix.dae
Joints:
- added joint gripper_link: type prismatic, parent e_link, child arm_gripper_link, origin xyz=0.0875 0 0 rpy=1.570796 0 0, axis 0 1 0, limit lower=0 upper=8 effort=0 velocity=0
- joint base_link_joint: axis 0 1 0 -> 0 -1 0; limit lower=-40 upper=0 effort=30 velocity=1 -> lower=0 upper=40 effort=30 velocity=1

File: public/urdf/rover/rover.urdf (robot description, URDF)
Before this commit: robot rover, 24 links, 23 joints
Links:
- added link arm_gripper_link; visual mesh filename=../meshes/arm_gripper_fix.dae
- link arm_a_link: mass 1 -> None; geometry visual mesh filename=../meshes/arm_a_fix.dae
- link arm_b_link: mass 1 -> None; geometry visual mesh filename=../meshes/arm_b_fix.dae
- link arm_base_link: mass None -> 3.0; geometry visual mesh filename=../meshes/rover_chassis.dae
- link arm_c_link: mass 1 -> None; geometry visual mesh filename=../meshes/arm_c_fix.dae
- link arm_d_link: mass 1 -> None; geometry visual mesh filename=../meshes/arm_d_fix.dae
- link arm_e_link: mass 1 -> None; geometry visual mesh filename=../meshes/arm_e_fix.dae
- link back_left_wheel_link: geometry collision cylinder length=0.08 radius=0.13; visual mesh filename=../meshes/rover_left_wheel.dae
- link back_right_wheel_link: geometry collision cylinder length=0.08 radius=0.13; visual mesh filename=../meshes/rover_right_wheel.dae
- link center_left_wheel_link: geometry collision cylinder length=0.08 radius=0.13; visual mesh filename=../meshes/rover_left_wheel.dae
- link center_right_wheel_link: geometry collision cylinder length=0.08 radius=0.13; visual mesh filename=../meshes/rover_right_wheel.dae
- link chassis_link: geometry collision box size=0.167 0.63 0.0891; collision box size=0.277 0.63 0.183
- link front_left_wheel_link: geometry collision cylinder length=0.08 radius=0.13; visual mesh filename=../meshes/rover_left_wheel.dae
- link front_right_wheel_link: geometry collision cylinder length=0.08 radius=0.13; visual mesh filename=../meshes/rover_right_wheel.dae
- link left_bogie_link: geometry collision box size=0.2 0.025 0.025; collision box size=0.2 0.025 0.025
- link left_rocker_link: geometry collision box size=0.2 0.025 0.025; collision box size=0.5 0.025 0.025
- link right_bogie_link: geometry collision box size=0.2 0.025 0.025; collision box size=0.2 0.025 0.025
- link right_rocker_link: geometry collision box size=0.2 0.025 0.025; collision box size=0.5 0.025 0.025
Joints:
- removed joint arm_a_link_to_arm_b_link
- removed joint arm_b_link_to_arm_c_link
- removed joint arm_c_link_to_arm_d_link
- removed joint arm_d_link_to_arm_e_link
- removed joint base_link_to_arm_base_link
- removed joint base_link_to_chassis_link
- removed joint chassis_link_to_arm_a_link
- removed joint chassis_link_to_left_gps
- removed joint chassis_link_to_left_rocker_link
- removed joint chassis_link_to_right_rocker_link
- removed joint left_bogie_link_to_center_left_wheel_link
- removed joint left_bogie_link_to_front_left_wheel_link
- removed joint left_rocker_link_to_back_left_wheel_link
- removed joint left_rocker_link_to_left_bogie_link
- removed joint right_bogie_link_to_center_right_wheel_link
- removed joint right_bogie_link_to_front_right_wheel_link
- removed joint right_rocker_link_to_back_right_wheel_link
- removed joint right_rocker_link_to_right_bogie_link
- added joint arm_a_to_arm_b: type revolute, parent arm_a_link, child arm_b_link, origin xyz=3.4348 -0.0005 4.9028 rpy=0 0 0, axis 0 1 0, limit lower=-0.7853981875 upper=0 effort=0 velocity=0
- added joint arm_b_to_arm_c: type revolute, parent arm_b_link, child arm_c_link, origin xyz=53.4363 0.0005 0.9052 rpy=0 0 0, axis 0 1 0, limit lower=-0.959931 upper=2.87979 effort=0 velocity=0
- added joint arm_c_to_arm_d: type revolute, parent arm_c_link, child arm_d_link, origin xyz=54.6037 0 8.8594 rpy=0 0 0, axis 0 1 0, limit lower=-2.35619 upper=2.35619 effort=0 velocity=0
- added joint arm_d_to_arm_e: type revolute, parent arm_d_link, child arm_e_link, origin xyz=4.488 0 0 rpy=0 0 0, axis 1 0 0, limit lower=-2.35619 upper=2.35619 effort=0 velocity=0
- added joint chassis_to_arm_a: type prismatic, parent chassis_link, child arm_a_link, origin xyz=16.4882 20.0235 49.1172 rpy=0 0 0, axis 0 -1 0, limit lower=0 upper=40 effort=0 velocity=0
- added joint gripper_link: type prismatic, parent arm_e_link, child arm_gripper_link, origin xyz=0.0875 0 0 rpy=1.570796 0 0, axis 0 1 0, limit lower=0 upper=8 effort=0 velocity=0
