Commit message: whoe rover done

File: public/urdf/rover/rover.urdf (robot description, URDF)
Before this commit: robot rover, 25 links, 11 joints
Links:
- removed link center_gps
- removed link imu
- removed link left_gps
- removed link long_range_camera_link
- removed link right_gps
- removed link zed_left_camera_frame
- link arm_base_link: mass 3.0 -> None
- link back_left_wheel_link: mass 3 -> None; geometry visual mesh filename=../meshes/rover_left_wheel_fix.dae
- link back_right_wheel_link: mass 3 -> None; geometry visual mesh filename=../meshes/rover_right_wheel_fix.dae
- link center_left_wheel_link: mass 3 -> None; geometry visual mesh filename=../meshes/rover_left_wheel_fix.dae
- link center_right_wheel_link: mass 3 -> None; geometry visual mesh filename=../meshes/rover_right_wheel_fix.dae
- link chassis_link: mass 15 -> None; geometry visual mesh filename=../meshes/rover_chassis.dae
- link front_left_wheel_link: mass 3 -> None; geometry visual mesh filename=../meshes/rover_left_wheel_fix.dae
- link front_right_wheel_link: mass 3 -> None; geometry visual mesh filename=../meshes/rover_right_wheel_fix.dae
- link left_bogie_link: mass 3 -> None; geometry visual mesh filename=../meshes/rover_left_bogie_fix.dae
- link left_rocker_link: mass 3 -> None; geometry visual mesh filename=../meshes/rover_left_rocker_fix.dae
- link right_bogie_link: mass 3 -> None; geometry visual mesh filename=../meshes/rover_right_bogie_fix.dae
- link right_rocker_link: mass 3 -> None; geometry visual mesh filename=../meshes/rover_right_rocker_fix.dae
Joints:
- removed joint chassis_link_to_center_gps
- removed joint chassis_link_to_imu
- removed joint chassis_link_to_long_range_camera_link
- removed joint chassis_link_to_right_gps
- removed joint chassis_link_to_zed_left_camera_frame
- added joint chassis_link_to_right_rocker_link: type revolute, parent chassis_link, child right_rocker_link, origin xyz=16.4665 -34.5164 41.3435 rpy=0 0 0, axis 0 1 0, limit lower=-0.122173 upper=0.523599
- added joint chassis_to_left_rocker: type revolute, parent chassis_link, child left_rocker_link, origin xyz=16.4665 34.5164 41.3435 rpy=0 0 0, axis 0 1 0, limit lower=-0.122173 upper=0.523599
- added joint left_bogie_to_center_left_wheel: type continuous, parent left_bogie_link, child center_left_wheel_link, origin xyz=-17.3532 9 -14.7659, axis 0 1 0, limit lower=-10 upper=10
- added joint left_bogie_to_front_left_wheel: type continuous, parent left_bogie_link, child front_left_wheel_link, origin xyz=21.5233 9 -14.7933, axis 0 1 0, limit lower=-10 upper=10
- added joint left_rocker_to_back_left_wheel: type continuous, parent left_rocker_link, child back_left_wheel_link, origin xyz=-41.7094 9 -28.513 , axis 0 1 0, limit lower=-10 upper=10
- added joint left_rocker_to_left_bogie: type revolute, parent left_rocker_link, child left_bogie_link, origin xyz=19.8948 0.0226 -13.8674 rpy=0 0 0, axis 0 1 0, limit lower=-0.349066 upper=0.349066
- added joint right_bogie_link_to_center_right_wheel_link: type continuous, parent right_bogie_link, child center_right_wheel_link, origin xyz=-17.3532 -9 -14.7659 rpy=0 0 0, axis 0 1 0, limit lower=-10 upper=10
- added joint right_bogie_link_to_front_right_wheel_link: type continuous, parent right_bogie_link, child front_right_wheel_link, origin xyz=21.5233 -9 -14.7933 rpy=0 0 0, axis 0 1 0, limit lower=-10 upper=10
- added joint right_rocker_link_to_back_right_wheel_link: type continuous, parent right_rocker_link, child back_right_wheel_link, origin xyz=-41.7094 -9 -28.513 rpy=0 0 0, axis 0 1 0, limit lower=-10 upper=10
- added joint right_rocker_link_to_right_bogie_link: type revolute, parent right_rocker_link, child right_bogie_link, origin xyz=19.8948 0.0226 -13.8674 rpy=0 0 0, axis 0 1 0, limit lower=-0.349066 upper=0.349066
- joint arm_a_to_arm_b: limit lower=-0.7853981875 upper=0 effort=0 velocity=0 -> lower=-0.7853981875 upper=0
- joint arm_b_to_arm_c: limit lower=-0.959931 upper=2.87979 effort=0 velocity=0 -> lower=-0.959931 upper=2.87979
- joint arm_c_to_arm_d: limit lower=-2.35619 upper=2.35619 effort=0 velocity=0 -> lower=-2.35619 upper=2.35619
- joint arm_d_to_arm_e: limit lower=-2.35619 upper=2.35619 effort=0 velocity=0 -> lower=-2.35619 upper=2.35619
- joint chassis_to_arm_a: limit lower=0 upper=40 effort=0 velocity=0 -> lower=0 upper=40
- joint gripper_link: limit lower=0 upper=8 effort=0 velocity=0 -> lower=0 upper=8

Commit message: home page progress

File: public/urdf/rover/rover.urdf (robot description, URDF)
Before this commit: robot rover, 19 links, 16 joints
Joints:
- removed joint chassis_link_to_right_rocker_link
- removed joint right_bogie_link_to_center_right_wheel_link
- removed joint right_bogie_link_to_front_right_wheel_link
- removed joint right_rocker_link_to_back_right_wheel_link
- removed joint right_rocker_link_to_right_bogie_link
- added joint chassis_to_right_rocker: type revolute, parent chassis_link, child right_rocker_link, origin xyz=16.4665 -34.5164 41.3435 rpy=0 0 0, axis 0 1 0, limit lower=-0.122173 upper=0.523599
- added joint right_bogie_to_center_right_wheel: type continuous, parent right_bogie_link, child center_right_wheel_link, origin xyz=-17.3532 -9 -14.7659 rpy=0 0 0, axis 0 1 0, limit lower=-10 upper=10
- added joint right_bogie_to_front_right_wheel: type continuous, parent right_bogie_link, child front_right_wheel_link, origin xyz=21.5233 -9 -14.7933 rpy=0 0 0, axis 0 1 0, limit lower=-10 upper=10
- added joint right_rocker_to_back_right_wheel: type continuous, parent right_rocker_link, child back_right_wheel_link, origin xyz=-41.7094 -9 -28.513 rpy=0 0 0, axis 0 1 0, limit lower=-10 upper=10
- added joint right_rocker_to_right_bogie: type revolute, parent right_rocker_link, child right_bogie_link, origin xyz=19.8948 0.0226 -13.8674 rpy=0 0 0, axis 0 1 0, limit lower=-0.349066 upper=0.349066

Commit message: astro port

File: public/urdf/rover/rover.urdf (robot description, URDF)
Before this commit: robot rover, 19 links, 16 joints
Links:
- link arm_a_link: geometry visual mesh filename=../meshes/arm_a_fix.glb
- link arm_b_link: geometry visual mesh filename=../meshes/arm_b_fix.glb
- link arm_base_link: geometry visual mesh filename=../meshes/rover_chassis.glb
- link arm_c_link: geometry visual mesh filename=../meshes/arm_c_fix.glb
- link arm_d_link: geometry visual mesh filename=../meshes/arm_d_fix.glb
- link arm_e_link: geometry visual mesh filename=../meshes/arm_e_fix.glb
- link arm_gripper_link: geometry visual mesh filename=../meshes/arm_gripper_fix.glb
- link back_left_wheel_link: geometry visual mesh filename=../meshes/rover_left_wheel_fix.glb
- link back_right_wheel_link: geometry visual mesh filename=../meshes/rover_right_wheel_fix.glb
- link center_left_wheel_link: geometry visual mesh filename=../meshes/rover_left_wheel_fix.glb
- link center_right_wheel_link: geometry visual mesh filename=../meshes/rover_right_wheel_fix.glb
- link chassis_link: geometry visual mesh filename=../meshes/rover_chassis.glb
- link front_left_wheel_link: geometry visual mesh filename=../meshes/rover_left_wheel_fix.glb
- link front_right_wheel_link: geometry visual mesh filename=../meshes/rover_right_wheel_fix.glb
- link left_bogie_link: geometry visual mesh filename=../meshes/rover_left_bogie_fix.glb
- link left_rocker_link: geometry visual mesh filename=../meshes/rover_left_rocker_fix.glb
- link right_bogie_link: geometry visual mesh filename=../meshes/rover_right_bogie_fix.glb
- link right_rocker_link: geometry visual mesh filename=../meshes/rover_right_rocker_fix.glb
